File: eagle/v0.80/aardvark-v0.80.brd (EAGLE design)
At the start: 100 x 98.9 mm, 28 parts, among them IC1 LM1117-3.3, J1 USB_MINI-B_SMT, U1 CH340C

Commit message: updated v0.80 w reset, boot, second schematic sheet
Parts:
- added C5: 100nF, rcl:C0805
- added Q1, Q2: (no value), SparkFun-DiscreteSemi:SOT23-3
- added R3, R4: 10k, rcl:R0805
- added S2: BOOT, SparkFun-Switches:TACTILE_SWITCH_SMD_6.0X3.5MM
- C3: value 4.7uF -> 100nF
Connections:
- new net !DTR: Q2.2, R3.2, U1.13
- new net !RTS: Q1.2, R4.2, U1.14
- new net N$10: Q1.1, R3.1
- new net N$11: Q2.1, R4.1
- net EN: now also Q1.3; no longer U1.14
- net GND: now also C5.2, S2.1
- net GP9: now also C5.1, Q2.3, S2.2; no longer U1.13
Routing:
- net GND: track 230.7 -> 0.00 mm, vias 2 -> 0
- net VCC: track 164.7 -> 0.00 mm, vias 2 -> 0
- net SDA: track 79.5 -> 0.00 mm
- net SCL: track 74.3 -> 0.00 mm
- net GP2: track 57.2 -> 0.00 mm, vias 1 -> 0
- net EN: track 48.5 -> 0.00 mm
- net TXO: track 38.0 -> 0.00 mm, vias 1 -> 0
- net RXI: track 34.1 -> 0.00 mm
- net UD+: track 31.8 -> 0.00 mm
- net UD-: track 31.7 -> 0.00 mm
- net GP9: track 31.5 -> 0.00 mm
- net VBUS: track 15.3 -> 0.00 mm, vias 2 -> 0
- net GP10: track 10.3 -> 0.00 mm
- net GP7: track 9.85 -> 0.00 mm
- net GP19: track 9.61 -> 0.00 mm
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Other:
- board text added: "DRAFT"
- board text added: "Triangle Embedded Interest Group Aardvarck 0.80 DRAFT ESP32-C3 + SLG47004V-DIP + Dialog SMD socket/program adapter"
- board text added: "Your ideas here"
- board text removed: "Triangle Embedded Interest Group Aardvarck 0.80 ESP32-C3 + SLG47004V-DIP + Dialog SMD socket/program adapter"

Commit message: example usage of v0.80 shown with aardvark-v0.80-board.pdf
Parts:
- moved FPGA1 5.08 mm to (37.8, 51.2)
- moved DIALOG-PGM 5.08 mm to (36.5, 56.3)
- moved SV1 5.08 mm to (27.6, 50.0)
- moved SV4 5.08 mm to (47.9, 50.0)
Other:
- board text added: "FOR INSTANCE A 25 AMP SSR"
- board text added: "Your ideas can modify to the left and add to the right to use up the whole board as needed."
- board text removed: "Your ideas here"

Commit message: proper momentary and power switches for v0.80
Parts:
- removed S1: RESET, SparkFun-Switches:TACTILE_SWITCH_SMD_6.0X3.5MM
- removed S2: BOOT, SparkFun-Switches:TACTILE_SWITCH_SMD_6.0X3.5MM
- added SP1, SP2: MTACT-SPST, CK-ATS2D1G_NC_LFS:MTACTSPST
- added SW1: CK_202011SCQN, CK_JS202011SCQN:CK_JS202011SCQN
- moved FD2 15.0 mm to (49.1, 71.9)
Connections:
- new net VOUT: C2.+, IC1.2, SW1.1-C
- net EN: now also SP1.PAD2; no longer S1.2
- net GND: now also SP1.PAD1, SP2.PAD1; no longer S1.1, S2.1
- net GP9: now also SP2.PAD2; no longer S2.2
- net VCC: now also SW1.1-NO; no longer C2.+, IC1.2
Routing:
- net GND: track 0.00 -> 242.6 mm, vias 0 -> 4
- net VCC: track 0.00 -> 158.3 mm
- net EN: track 0.00 -> 139.8 mm, vias 0 -> 2
- net GP9: track 0.00 -> 126.6 mm, vias 0 -> 2
- net SDA: track 0.00 -> 76.0 mm
- net SCL: track 0.00 -> 69.7 mm
- net GP2: track 0.00 -> 55.1 mm
- net !DTR: track 0.00 -> 53.3 mm, vias 0 -> 2
- net !RTS: track 0.00 -> 50.8 mm, vias 0 -> 2
- net TXO: track 0.00 -> 38.0 mm
- net RXI: track 0.00 -> 34.1 mm
- net UD+: track 0.00 -> 31.5 mm
- net UD-: track 0.00 -> 27.6 mm, vias 0 -> 2
- net VBUS: track 0.00 -> 15.7 mm
- net VOUT: track 0.00 -> 12.9 mm
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