File: eagle/v0.80/aardvark-v0.80.brd (EAGLE design)
At the start: 25.4 x 88.9 mm, 27 parts, among them IC1 LM1117-3.3, J1 MINI, U1 CH340C

Commit message: eagle/v0.80/{*.brd,sch} added part numbers
Parts:
- C2: value 10uF -> 10uF 399-6674-1-ND
Changed lines of the file:
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@@
 <attribute name="POPULARITY" value="49" x="13.29" y="84.05" size="1.778" layer="27" display="off"/>
 </element>
-<element name="C2" library="rcl" library_urn="urn:adsk.eagle:library:334" package="C0805" package3d_urn="urn:adsk.eagle:package:23617/2" value="10uF" x="12.286" y="78.024" smashed="yes" rot="R180">
+<element name="C2" library="rcl" library_urn="urn:adsk.eagle:library:334" package="C0805" package3d_urn="urn:adsk.eagle:package:23617/2" value="10uF 399-6674-1-ND" x="12.286" y="78.024" smashed="yes" rot="R180">
 <attribute name="NAME" x="16.096" y="78.659" size="1.016" layer="25" font="vector" ratio="20" rot="R180"/>
 <attribute name="POPULARITY" value="63" x="12.286" y="78.024" size="1.778" layer="27" rot="R180" display="off"/>
