File: eagle/v0.70/aardvark-v0.70.brd (EAGLE design)
At the start: 25.4 x 88.9 mm, 22 parts, among them IC1 LM1117-3.3, J1 USB_MINI-B_SMT, U1 CH340C

Commit message: aardvark v0.70 as shipped to OSH Park
Parts:
- moved FD2 66.7 mm to (23.6, 64.9)
- moved FD1 19.7 mm to (4.38, 87.6)
Connections:
- net SCL: now also SV2.4; no longer SV2.3
- net SDA: now also SV2.3; no longer SV2.4
Routing:
- net EN: track 85.6 -> 49.8 mm, vias 1 -> 2
- net GND: track 138.2 -> 123.4 mm, vias 1 -> 2
- net VCC: track 134.7 -> 149.2 mm, vias 2 -> 1
- net SDA: track 77.4 -> 69.4 mm
- net TXO: track 34.5 -> 39.5 mm, vias 1 -> 2
- net VBUS: track 12.6 -> 14.2 mm, vias 2 -> 0
- net GP9: track 28.2 -> 27.1 mm, vias 2 -> 3
- net SCL: track 75.5 -> 76.4 mm

Commit message: Finished initial ECOs for 0.70 board
Parts:
- added C4, C5: 100nF, rcl:C0805
- added Q1, Q2: (no value), SparkFun-DiscreteSemi:SOT23-3
- added R3, R4: 10k, rcl:R0805
- added S2: RESET, SparkFun-Switches:TACTILE_SWITCH_SMD_6.0X3.5MM
- C3: value 4.7uF -> 100nF
Connections:
- new net !DTR: Q2.2, R3.2
- new net !RTS: Q1.2, R4.2
- new net N$10: Q1.1, R3.1
- new net N$11: Q2.1, R4.1
- net EN: now also Q1.3
- net GND: now also C4.2, C5.1, S2.1
- net GP9: now also C4.1, Q2.3, S2.2
- net TXO: now also C5.2, U1.16, U1.4
- net VCC: no longer U1.16, U1.4
Routing:
- net VCC: track 149.2 -> 141.7 mm
- net TXO: track 39.5 -> 46.6 mm
